File: Macropad/Macropad.kicad_pcb (KiCad board)
At the start: 2 copper layers, 112.2 x 163 mm, 122 parts, among them J201 TSOP4838_C124647, J202 IR_LED_TX_HDR, J301 LED_CHAIN, J302 LCD_SPI_PWRDATA, J303 LCD_SPI_CTRL, J304 TOUCH_I2C_SD_IRQ, J400 BATTERY_LIPO, J401 BAT_CHG_BOOST, J402 USB_C_CHG_IN, Q501 AO3400A, SW1 SW_Push, SW10 SW_Push, SW11 SW_Push, SW12 SW_Push, SW13 SW_Push, SW14 SW_Push, SW15 SW_Push, SW16 SW_Push, SW17 SW_Push, SW18 SW_Push, SW19 SW_Push, SW2 SW_Push, SW20 SW_Push, SW21 SW_Push, SW22 SW_Push, SW23 SW_Push, SW24 SW_Push, SW25 SW_Push, SW26 SW_Push, SW3 SW_Push, SW4 SW_Push, SW401 RotaryEncoder_Switch, SW402 SW_Push, SW5 SW_Push, SW6 SW_Push, SW7 SW_Push, SW8 SW_Push, SW9 SW_Push, U402 AP7361C-33E, U403 MCP73831, U404 MT3608, U901 ESP32-S3-WROOM-1-N8R8

Commit message: Board and firmware updates
Connections:
- U901 pad 13: (no net) -> USB_DN
- U901 pad 14: TOUCH_INT -> USB_DP
- U901 pad 16: (no net) -> TOUCH_INT
Routing:
- net USB_DP: track 0.00 -> 31.0 mm
- net USB_DN: track 0.00 -> 30.6 mm
- net 5V_SYS: track 1533.3 -> 1545.7 mm
- net TOUCH_INT: track 51.1 -> 52.7 mm
- added copper zone on B.Cu, net GND
- added copper zone on F.Cu, net GND
Changed lines of the file:
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@@
 	(net 97 "VBUS")
 	(net 98 "TOUCH_INT")
+	(net 99 "USB_DN")
+	(net 100 "USB_DP")
 	(footprint "C_0603_1608Metric_LOCAL"
 		(layer "F.Cu")
@@
 			(net 23 "GND")
 		)
+		(pad "A6" smd roundrect
+			(at 0.75 -3.08)
+			(size 0.3 1.2)
+			(layers "F.Cu" "F.Mask" "F.Paste")
+			(roundrect_rratio 0.25)
+			(net 100 "USB_DP")
+		)
+		(pad "A7" smd roundrect
+			(at -0.75 -3.08)
+			(size 0.3 1.2)
+			(layers "F.Cu" "F.Mask" "F.Paste")
+			(roundrect_rratio 0.25)
+			(net 99 "USB_DN")
+		)
 		(pad "B5" smd roundrect
 			(at 0.5 -3.08 180)
@@
 			(net 52 "USB_CC2")
 		)
+		(pad "B6" smd roundrect
+			(at 0.75 -3.08)
+			(size 0.3 1.2)
+			(layers "F.Cu" "F.Mask" "F.Paste")
+			(roundrect_rratio 0.25)
+			(net 100 "USB_DP")
+		)
+		(pad "B7" smd roundrect
+			(at -0.75 -3.08)
+			(size 0.3 1.2)
+			(layers "F.Cu" "F.Mask" "F.Paste")
+			(roundrect_rratio 0.25)
+			(net 99 "USB_DN")
+		)
 		(pad "B9" smd roundrect
 			(at -1.52 -3.08)
@@
 			(size 1.5 0.9)
 			(layers "F.Cu" "F.Mask" "F.Paste")
+			(net 99 "USB_DN")
 		)
 		(pad "14" smd rect
@@
 			(size 1.5 0.9)
 			(layers "F.Cu" "F.Mask" "F.Paste")
-			(net 98 "TOUCH_INT")
+			(net 100 "USB_DP")
 		)
 		(pad "15" smd rect
@@
 			(size 1.5 0.9)
 			(layers "F.Cu" "F.Mask" "F.Paste")
+			(net 98 "TOUCH_INT")
 		)
 		(pad "17" smd rect
@@
 		(layer "Edge.Cuts")
 	)
+	(zone
+		(net 23)
+		(net_name "GND")
+		(layer "F.Cu")
+		(name "GND_FLOOD_TOP")
+		(hatch edge 0.5)
+		(priority 0)
+		(connect_pads
+			(clearance 0.2)
+		)
+		(min_thickness 0.2)
+		(filled_areas_thickness no)
+		(fill yes
+			(thermal_gap 0.3)
+			(thermal_bridge_width 0.3)
+		)
+		(polygon
+			(pts
+				(xy -5 -41)
+				(xy 107.25 -41)
+				(xy 107.25 122)
+				(xy -5 122)
+			)
+		)
+	)
+	(zone
+		(net 23)
+		(net_name "GND")
+		(layer "B.Cu")
+		(name "GND_FLOOD_BOTTOM")
+		(hatch edge 0.5)
+		(priority 0)
+		(connect_pads
+			(clearance 0.2)
+		)
+		(min_thickness 0.2)
+		(filled_areas_thickness no)
+		(fill yes
+			(thermal_gap 0.3)
+			(thermal_bridge_width 0.3)
+		)
+		(polygon
+			(pts
+				(xy -5 -41)
+				(xy 107.25 -41)
+				(xy 107.25 122)
+				(xy -5 122)
+			)
+		)
+	)
 	(segment
 		(start 105.25 6.985)
@@
 	(segment
 		(start 55.945 -39.08)
+		(end 86 -45)
+		(width 0.3)
+		(layer "F.Cu")
+		(net 22)
+	)
+	(segment
+		(start 86 -45)
 		(end 92.25 -25.46)
 		(width 0.3)
@@
 	)
 	(segment
-		(start 66.5 -11.75)
+		(start 69.535 -10.5)
 		(end 66.5 -24)
 		(width 0.25)
@@
 		(net 98)
 	)
+	(segment
+		(start 66.5 -11.75)
+		(end 51.875 -39.08)
+		(width 0.2)
+		(layer "F.Cu")
+		(net 100)
+	)
+	(segment
+		(start 66.5 -13.02)
+		(end 50.375 -39.08)
+		(width 0.2)
+		(layer "F.Cu")
+		(net 99)
+	)
+	(zone
+		(net 0)
+		(net_name "")
+		(layers "F.Cu" "B.Cu")
+		(name "U901_ANT_KEEP_OUT")
+		(hatch edge 0.5)
+		(priority 1)
+		(connect_pads
+			(clearance 0)
+		)
+		(min_thickness 0.25)
+		(filled_areas_thickness no)
+		(keepout
+			(tracks not_allowed)
+			(vias not_allowed)
+			(pads not_allowed)
+			(copperpour not_allowed)
+		)
+		(polygon
+			(pts
+				(xy 73.5 -42)
+				(xy 85 -42)
+				(xy 85 -32.5)
+				(xy 73.5 -32.5)
+			)
+		)
+	)
 	(embedded_fonts no)

Commit message: updates
Parts:
- J303: footprint GEN_PinHeader_1x5_P2.54 -> GEN_PinHeader_1x4_P2.54
- moved J304 8.40 mm to (56.9, -6.50), turned to 0 degrees
- moved J302 7.73 mm to (44.2, -6.50), turned to 0 degrees
- moved J303 7.46 mm to (34.2, -6.50), turned to 0 degrees
- turned J301 to 0 degrees
- turned J401 to 0 degrees
Connections:
- J302 pad 3: LCD_MOSI -> LCD_SCLK
- J302 pad 4: LCD_SCLK -> LCD_MOSI
- J303 pad 1: LCD_CS -> SPI_MISO
- J303 pad 2: LCD_DC -> LCD_CS
- J303 pad 3: LCD_RST -> LCD_DC
- J303 pad 4: LCD_BL -> LCD_RST
- J304 pad 1: TOUCH_SDA -> LCD_BL
- J304 pad 2: SPI_MISO -> TOUCH_INT
- J304 pad 3: TOUCH_SCL -> TOUCH_SDA
- J304 pad 4: SD_CS -> TOUCH_SCL
- J304 pad 5: TOUCH_INT -> SD_CS
Routing:
- net LCD_BL: track 144.8 -> 109.9 mm
- net TOUCH_INT: track 52.7 -> 42.1 mm
- net LCD_SCLK: track 89.2 -> 79.4 mm
- net SPI_MISO: track 60.3 -> 70.0 mm
- net TOUCH_SCL: track 67.7 -> 60.7 mm
- net SD_CS: track 77.7 -> 70.8 mm
- net 3V3: track 444.7 -> 437.9 mm
- net LCD_MOSI: track 84.0 -> 79.0 mm
- net LCD_CS: track 127.5 -> 122.8 mm
- net LCD_DC: track 130.7 -> 126.0 mm
- net TOUCH_SDA: track 49.1 -> 44.4 mm
- net LCD_RST: track 136.5 -> 131.8 mm
Other:
- board text added: "3Vo"
- board text added: "CCS"
- board text added: "CLK"
- board text added: "CS"
- board text added: "D/C"
- board text added: "GND"
- board text added: "IRQ"
- board text added: "Lite"
- board text added: "MISO"
- board text added: "MOSI"
- board text added: "RST"
- board text added: "SCL"
- board text added: "SDA"
