File: Macropad/__layer_test.kicad_pcb (KiCad board)
At the start: 4 copper layers, 116.2 x 163 mm, 122 parts, among them J201 TSOP4838_C124647, J202 IR_LED_TX_HDR, J301 LED_CHAIN, J302 LCD_SPI_PWRDATA, J303 LCD_SPI_CTRL, J304 TOUCH_I2C_SD_IRQ, J400 BATTERY_LIPO, J401 BAT_CHG_BOOST, J402 USB_C_CHG_IN, Q501 AO3400A, SW1 SW_Push, SW10 SW_Push, SW11 SW_Push, SW12 SW_Push, SW13 SW_Push, SW14 SW_Push, SW15 SW_Push, SW16 SW_Push, SW17 SW_Push, SW18 SW_Push, SW19 SW_Push, SW2 SW_Push, SW20 SW_Push, SW21 SW_Push, SW22 SW_Push, SW23 SW_Push, SW24 SW_Push, SW25 SW_Push, SW26 SW_Push, SW3 SW_Push, SW4 SW_Push, SW401 RotaryEncoder_Switch, SW402 MSS-102545-14A-V-SMT, SW402 SW_Push, SW5 SW_Push, SW6 SW_Push, SW7 SW_Push, SW8 SW_Push, SW9 SW_Push, U402 AP7361C-33E, U403 MCP73831, U404 MT3608, U901 ESP32-S3-WROOM-1-N8R8

Commit message: Updates
Routing:
- net 5V_SYS: vias 29 -> 30
